File: hardware/fmcw3.kicad_pcb (KiCad board)
At the start: 4 copper layers, 101.8 x 46.8 mm, 429 parts, among them CON1 SD_Card_DM3BT, CON2 BARREL_JACK, P1 SMA, P10 CONN_01X01, P11 CONN_01X01, P12 CONN_01X01, P13 CONN_01X01, P14 CONN_01X01, P15 CONN_01X01, P16 CONN_01X01, P2 SMA, P3 CONN_02X04, P4 CONN_02X04, P5 CONN_01X01, P6 CONN_01X01, P7 CONN_01X01, P8 CONN_01X01, P9 CONN_01X01, Q1 RE1C002UN, Q2 DNP(RE1C002UN), SW2 SW_PUSH, U1 ADF4158, U10 HMC431LP4, U11 SKY65404, U12 PAT1220-6dB, U13 TRF37A73, U14 MGA-25203, U15 SMA, U16 SKY65404, U17 L7980, U18 L7980, U19 L7980, U2 LP5907-1.8, U20 LP5907-3.0, U21 LP2985A-10DBVR, U22 TPS7A91, U23 TPS7A91, U24 TPS7A91, U25 MIC5301-3.3, U26 5400BL15B050E, U27 5400BL15B050E, U28 5400BL15B050E, U29 ADL5802, U3 PAT1220-6dB, U30 XC7A15T-1FTG256C, U31 USB-MICRO, U32 93LC46B, U33 FT2232H, U34 ADA4940-2, U35 ADA4940-2, U39 LP5907-3.0, U4 KT2520K, U40 W25Q32JV, U5 NC7S04P5X, U6 NB3N551, U7 TLV172DCK, U8 LTC2292, U9 TRF37A73, Y1 ABM10-167-12.000MHZ-T3

Commit message: Migrate KiCad 4 project to KiCad 10
Converts the 2017-era project (EESchema Schematic File Version 2,
kicad_pcb 20170123) to KiCad 10 format (version 20260306).

Schematics could not be converted by any kicad-cli: KiCad 10 dropped the
legacy EESchema reader, and KiCad 8's CLI has no upgrade subcommand. The
conversion ran through the KiCad 8 GUI (docker kicad/kicad:8.0), then
kicad-cli sch upgrade locally for each sheet.

- Symbol remap + rescue: 657 symbols resolved, 0 failures. 607 mapped to
  fmcw3-rescue (generic parts pinned to the 2017 cache so pin numbering
  does not silently change), 50 to the project library.
- sym-lib-table and fmcw3-rescue.lib are load-bearing: without them the
  rescued symbols do not resolve on another machine.
- Fixed Sheetfile properties in the root sheet, which the GUI conversion
  left pointing at the old .sch names; only the top sheet loaded until
  then. Hierarchy now resolves: 437 components, 406 nets, no duplicate
  or unannotated refs (both rx.sch instances survived distinctly).
- kicad-cli sch upgrade only converts the file named, not the hierarchy,
  so each subsheet was upgraded individually.

PCB converted with a "legacy zone fill strategy is not supported anymore"
warning -- copper must be re-poured and DRC re-run before it is trusted.

imu.sch is retained as legacy: it is an orphan sheet, not instantiated in
the hierarchy, so the GUI never converted it. It has no replacement here.

Original legacy project remains intact on master.

Co-Authored-By: Claude Opus 5 <noreply@anthropic.com>
Other:
- net class Default removed
