File: hardware/adc.kicad_sch (KiCad schematic)
At the start: 38 parts, among them U39 LP5907-3.0, U8 LTC2292

Commit message: Hardware: apply sourcing fields to fmcw3 schematic symbols (hw-02)
Adds Manufacturer, MPN, DigiKey PN, Status (obsolete/NFND/needs-David:
see docs/hardware/fmcw3 memo) and, for generic passives, spec-only
Tolerance/Voltage/Dielectric hidden fields to 355 refs from
parts/fields_to_apply.csv. The 4 existing manf# fields are renamed to
MPN. Value, footprint, nets and PCB untouched. ERC 679 unchanged;
netlist nets/components identical.

Directive: hw-02
Tracker: #58

Co-Authored-By: Claude Opus 5.5 <noreply@anthropic.com>
Parts:
- C163, C164, C165, C166, C167, C168, C19, C20, C216, C217, C218, C219, C22, C220, C221, C23, C30, C31: Dielectric (none) -> unspecified; Tolerance (none) -> unspecified; Voltage (none) -> >=6.3 V (inferred default: no supply rail on these nets)
- C222, C249: Dielectric (none) -> unspecified; Tolerance (none) -> unspecified; Voltage (none) -> >=6.3 V (inferred: 3 V on 3V0)
- C223, C224, C225, C24, C248, C25, C27: Dielectric (none) -> unspecified; Tolerance (none) -> unspecified; Voltage (none) -> >=6.3 V (inferred: 3.6 V on 3V6)
- R100, R20, R21, R91, R93, R97, R98, R99: Tolerance (none) -> unspecified
- U39: DigiKey PN (none) -> 296-40357-1-ND; MPN (none) -> LP5907MFX-3.0/NOPB; Manufacturer (none) -> Texas Instruments
- U8: Status (none) -> needs-David: see docs/hardware/fmcw3 memo
