File: hardware/fmcw3.kicad_sch (KiCad schematic)
At the start: 20 parts, among them P5 CONN_01X01, P7 CONN_01X01, P8 CONN_01X01, U2 LP5907-1.8, U4 KT2520K, U5 NC7S04P5X, U6 NB3N551

Commit message: Hardware: apply sourcing fields to fmcw3 schematic symbols (hw-02)
Adds Manufacturer, MPN, DigiKey PN, Status (obsolete/NFND/needs-David:
see docs/hardware/fmcw3 memo) and, for generic passives, spec-only
Tolerance/Voltage/Dielectric hidden fields to 355 refs from
parts/fields_to_apply.csv. The 4 existing manf# fields are renamed to
MPN. Value, footprint, nets and PCB untouched. ERC 679 unchanged;
netlist nets/components identical.

Directive: hw-02
Tracker: #58

Co-Authored-By: Claude Opus 5.5 <noreply@anthropic.com>
Parts:
- C12: Dielectric (none) -> unspecified; Tolerance (none) -> unspecified; Voltage (none) -> >=6.3 V (inferred: 3 V on 3V0)
- C13, C16: Dielectric (none) -> unspecified; Tolerance (none) -> unspecified; Voltage (none) -> >=6.3 V (inferred default: no supply rail on these nets)
- C15, C17, C9: Dielectric (none) -> unspecified; Tolerance (none) -> unspecified; Voltage (none) -> >=6.3 V (inferred: 3.6 V on 3V6)
- FB1: DigiKey PN (none) -> 490-5263-1-ND; MPN (none) -> BLM18PG181SN1D; Manufacturer (none) -> Murata Electronics
- R13, R15, R16, R3, R8: Tolerance (none) -> unspecified
- U2: DigiKey PN (none) -> 296-41463-1-ND; MPN (none) -> LP5907MFX-1.8/NOPB; Manufacturer (none) -> Texas Instruments
- U4: Status (none) -> needs-David: see docs/hardware/fmcw3 memo
- U5: DigiKey PN (none) -> NC7S04P5XCT-ND; MPN (none) -> NC7S04P5X; Manufacturer (none) -> onsemi
- U6: DigiKey PN (none) -> NB3N551MNR4GOSCT-ND; MPN (none) -> NB3N551MNR4G; Manufacturer (none) -> onsemi; Status (none) -> Obsolete: see docs/hardware/fmcw3 memo
