File: hardware/fpga.kicad_sch (KiCad schematic)
At the start: 66 parts, among them CON1 SD_Card_DM3BT, P10 CONN_01X01, P11 CONN_01X01, P12 CONN_01X01, P13 CONN_01X01, P14 CONN_01X01, P15 CONN_01X01, P16 CONN_01X01, P3 CONN_02X04, P4 CONN_02X04, P6 CONN_01X01, P9 CONN_01X01, Q2 DNP(RE1C002UN), SW2 SW_PUSH, U30A XC7A15T-1FTG256C, U30B XC7A15T-1FTG256C, U30C XC7A15T-1FTG256C, U30D XC7A15T-1FTG256C, U30E XC7A15T-1FTG256C, U30F XC7A15T-1FTG256C, U30G XC7A15T-1FTG256C, U40 W25Q32JV

Commit message: Hardware: apply sourcing fields to fmcw3 schematic symbols (hw-02)
Adds Manufacturer, MPN, DigiKey PN, Status (obsolete/NFND/needs-David:
see docs/hardware/fmcw3 memo) and, for generic passives, spec-only
Tolerance/Voltage/Dielectric hidden fields to 355 refs from
parts/fields_to_apply.csv. The 4 existing manf# fields are renamed to
MPN. Value, footprint, nets and PCB untouched. ERC 679 unchanged;
netlist nets/components identical.

Directive: hw-02
Tracker: #58

Co-Authored-By: Claude Opus 5.5 <noreply@anthropic.com>
Parts:
- C170, C171, C182, C183, C184, C185, C186, C187, C188, C189, C190, C191, C192, C193, C194, C195, C196, C197, C198, C199, C200, C201, C202, C203, C204, C205, C250, C251: Dielectric (none) -> unspecified; Tolerance (none) -> unspecified; Voltage (none) -> >=6.3 V (inferred: 3.3 V on 3V3D)
- C18, C252: Dielectric (none) -> unspecified; Tolerance (none) -> unspecified; Voltage (none) -> >=6.3 V (inferred: 3.6 V on 3V6)
- C181: Dielectric (none) -> unspecified; Tolerance (none) -> unspecified; Voltage (none) -> >=6.3 V (inferred: 1 V on 1V0)
- CON1: DigiKey PN (none) -> HR1942CT-ND; MPN (none) -> DM3BT-DSF-PEJS; Manufacturer (none) -> Hirose Electric Co Ltd
- D6, P3, P4: Tolerance (none) -> n/a
- R109, R111, R112, R114, R115, R117, R118, R130, R70: Tolerance (none) -> unspecified
- SW2: DigiKey PN (none) -> P16850TR-ND; MPN (none) -> EVP-AWBA2A; Manufacturer (none) -> Panasonic Industry; Status (none) -> Obsolete: see docs/hardware/fmcw3 memo
- U30A, U30B, U30C, U30D, U30E, U30F, U30G: DigiKey PN (none) -> 122-1930-ND; MPN (none) -> XC7A15T-1FTG256C; Manufacturer (none) -> AMD
- U40: DigiKey PN (none) -> 256-W25Q32JVZPIQ-TUBE-ND; MPN (none) -> W25Q32JVZPIQ; Manufacturer (none) -> Winbond Electronics; Status (none) -> Obsolete: see docs/hardware/fmcw3 memo
