File: hardware/if.kicad_sch (KiCad schematic)
At the start: 61 parts, among them U34A ADA4940-2, U34B ADA4940-2, U35A ADA4940-2, U35B ADA4940-2

Commit message: Hardware: apply sourcing fields to fmcw3 schematic symbols (hw-02)
Adds Manufacturer, MPN, DigiKey PN, Status (obsolete/NFND/needs-David:
see docs/hardware/fmcw3 memo) and, for generic passives, spec-only
Tolerance/Voltage/Dielectric hidden fields to 355 refs from
parts/fields_to_apply.csv. The 4 existing manf# fields are renamed to
MPN. Value, footprint, nets and PCB untouched. ERC 679 unchanged;
netlist nets/components identical.

Directive: hw-02
Tracker: #58

Co-Authored-By: Claude Opus 5.5 <noreply@anthropic.com>
Parts:
- C126, C127: Dielectric (none) -> unspecified; Tolerance (none) -> unspecified; Voltage (none) -> >=10 V (inferred: 5 V on Net-(C126-Pad1))
- C128, C129, C130, C131: Dielectric (none) -> unspecified; Tolerance (none) -> unspecified; Voltage (none) -> >=10 V (inferred: 5 V on 5V)
- C132, C133, C134, C135, C136, C137: Dielectric (none) -> unspecified; Tolerance (none) -> unspecified; Voltage (none) -> >=6.3 V (inferred default: no supply rail on these nets)
- C138, C139, C150, C151: Dielectric (none) -> unspecified; Tolerance (none) -> unspecified; Voltage (none) -> >=6.3 V (inferred: 3.6 V on 3V6)
- L10, L11, L8, L9, R55, R56, R57, R58, R59, R60, R61, R62, R87, R89, R90, R94: Tolerance (none) -> unspecified
- U34A, U34B, U35A, U35B: DigiKey PN (none) -> 505-ADA4940-2ACPZ-R7CT-ND; MPN (none) -> ADA4940-2ACPZ-R7; Manufacturer (none) -> Analog Devices Inc.
