File: hardware/mixer.kicad_sch (KiCad schematic)
At the start: 31 parts, among them U26 5400BL15B050E, U27 5400BL15B050E, U28 5400BL15B050E, U29 ADL5802

Commit message: Hardware: apply sourcing fields to fmcw3 schematic symbols (hw-02)
Adds Manufacturer, MPN, DigiKey PN, Status (obsolete/NFND/needs-David:
see docs/hardware/fmcw3 memo) and, for generic passives, spec-only
Tolerance/Voltage/Dielectric hidden fields to 355 refs from
parts/fields_to_apply.csv. The 4 existing manf# fields are renamed to
MPN. Value, footprint, nets and PCB untouched. ERC 679 unchanged;
netlist nets/components identical.

Directive: hw-02
Tracker: #58

Co-Authored-By: Claude Opus 5.5 <noreply@anthropic.com>
Parts:
- C108, C115, C116, C120, C121, C122, C123: Dielectric (none) -> unspecified; Tolerance (none) -> unspecified; Voltage (none) -> >=10 V (inferred: 5 V on Net-(U1-VP))
- C109, C110, C111, C112, C113, C114: Dielectric (none) -> unspecified; Status (none) -> needs-David: see docs/hardware/fmcw3 memo; Tolerance (none) -> unspecified; Voltage (none) -> >=6.3 V (inferred default: no supply rail on these nets)
- C117, C118, C119: Dielectric (none) -> unspecified; Tolerance (none) -> unspecified; Voltage (none) -> >=10 V (inferred: 5 V on 5VF)
- C162: Dielectric (none) -> unspecified; Tolerance (none) -> unspecified; Voltage (none) -> >=10 V (inferred: 5.6 V on 5V6)
- FB13: DigiKey PN (none) -> 490-5263-1-ND; MPN (none) -> BLM18PG181SN1D; Manufacturer (none) -> Murata Electronics
- R49, R51, R52, R53, R54: Tolerance (none) -> unspecified
- U26, U27, U28: DigiKey PN (none) -> 712-5400BL15B0050001ECT-ND; MPN (none) -> 5400BL15B0050001E; Manufacturer (none) -> Johanson Technology Inc.
- U29: DigiKey PN (none) -> ADL5802ACPZ-R7CT-ND; MPN (none) -> ADL5802ACPZ-R7; Manufacturer (none) -> Analog Devices Inc.
