File: hardware/power.kicad_sch (KiCad schematic)
At the start: 96 parts, among them CON2 BARREL_JACK, U17 L7980, U18 L7980, U19 L7980, U20 LP5907-3.0, U21 LP2985A-10DBVR, U22 TPS7A91, U23 TPS7A91, U24 TPS7A91, U25 MIC5301-3.3

Commit message: Hardware: apply sourcing fields to fmcw3 schematic symbols (hw-02)
Adds Manufacturer, MPN, DigiKey PN, Status (obsolete/NFND/needs-David:
see docs/hardware/fmcw3 memo) and, for generic passives, spec-only
Tolerance/Voltage/Dielectric hidden fields to 355 refs from
parts/fields_to_apply.csv. The 4 existing manf# fields are renamed to
MPN. Value, footprint, nets and PCB untouched. ERC 679 unchanged;
netlist nets/components identical.

Directive: hw-02
Tracker: #58

Co-Authored-By: Claude Opus 5.5 <noreply@anthropic.com>
Parts:
- C100, C79, C82, C83, C84, C86: Dielectric (none) -> unspecified; Tolerance (none) -> unspecified; Voltage (none) -> >=10 V (inferred: 5.6 V on 5V6)
- C101, C102, C106, C76, C77, C78, C80, C85, C87, C88, C93, C94: Dielectric (none) -> unspecified; Tolerance (none) -> unspecified; Voltage (none) -> >=6.3 V (inferred: 3.6 V on 3V6)
- C60, C61, C62, C64, C70, C89: Dielectric (none) -> unspecified; Tolerance (none) -> unspecified; Voltage (none) -> >=25 V (inferred: 15 V on 12V)
- C63, C65, C66, C67, C68, C69, C90, C91, C92, C95: Dielectric (none) -> unspecified; Tolerance (none) -> unspecified; Voltage (none) -> >=6.3 V (inferred default: no supply rail on these nets)
- C73: Dielectric (none) -> unspecified; Tolerance (none) -> unspecified; Voltage (none) -> >=6.3 V (inferred: 1 V on Net-(C73-Pad1))
- C74: Dielectric (none) -> unspecified; Tolerance (none) -> unspecified; Voltage (none) -> >=6.3 V (inferred: 3.6 V on Net-(C74-Pad1))
- C75: Dielectric (none) -> unspecified; Tolerance (none) -> unspecified; Voltage (none) -> >=10 V (inferred: 5.6 V on Net-(C75-Pad1))
- C96: Dielectric (none) -> unspecified; Tolerance (none) -> unspecified; Voltage (none) -> >=10 V (inferred: 5 V on 5V)
- C97, C99: Dielectric (none) -> unspecified; Tolerance (none) -> unspecified; Voltage (none) -> >=6.3 V (inferred: 3.3 V on 3V3A)
- C98: Dielectric (none) -> unspecified; Tolerance (none) -> unspecified; Voltage (none) -> >=16 V (inferred: 10 V on 10V)
- CON2: DigiKey PN (none) -> EJ508A-ND; MPN (none) -> EJ508A; Manufacturer (none) -> MPD (Memory Protection Devices)
- D1: Tolerance (none) -> n/a
- D2, D3, D4: DigiKey PN (none) -> 2832-SS13FLTR-ND; MPN (none) -> SS13FL; Manufacturer (none) -> onsemi; Status (none) -> Obsolete: see docs/hardware/fmcw3 memo
- FB11: DigiKey PN (none) -> 1276-6374-2-ND; MPN (none) -> CIC21P101NE; Manufacturer (none) -> Samsung Electro-Mechanics; Status (none) -> Obsolete: see docs/hardware/fmcw3 memo
- L5, L6, L7: DigiKey PN (none) -> SRR6040A-330MCT-ND; MPN (none) -> SRR6040A-330M; Manufacturer (none) -> Bourns Inc.; Status (none) -> NFND: see docs/hardware/fmcw3 memo
- R103, R104, R24, R25, R26, R27, R28, R29, R30, R32, R33, R34, R35, R36, R37, R38, R41, R42, R43, R44, R45, R46, R47, R48: Tolerance (none) -> unspecified
- U17, U18, U19: DigiKey PN (none) -> 497-10813-1-ND; MPN (none) -> L7980TR; Manufacturer (none) -> STMicroelectronics
- U20: DigiKey PN (none) -> 296-40357-1-ND; MPN (none) -> LP5907MFX-3.0/NOPB; Manufacturer (none) -> Texas Instruments
- U21: DigiKey PN (none) -> 296-24264-1-ND; MPN (none) -> LP2985A-10DBVR; Manufacturer (none) -> Texas Instruments
- U22, U23, U24: DigiKey PN (none) -> 296-45298-1-ND; MPN (none) -> TPS7A9101DSKT; Manufacturer (none) -> Texas Instruments
- U25: DigiKey PN (none) -> 576-2840-1-ND; MPN (none) -> MIC5301-3.3YD5-TR; Manufacturer (none) -> Microchip Technology
