File: hardware/rx.kicad_sch (KiCad schematic)
At the start: 19 parts, among them P1 SMA, U11 SKY65404, U9 TRF37A73

Commit message: Hardware: apply sourcing fields to fmcw3 schematic symbols (hw-02)
Adds Manufacturer, MPN, DigiKey PN, Status (obsolete/NFND/needs-David:
see docs/hardware/fmcw3 memo) and, for generic passives, spec-only
Tolerance/Voltage/Dielectric hidden fields to 355 refs from
parts/fields_to_apply.csv. The 4 existing manf# fields are renamed to
MPN. Value, footprint, nets and PCB untouched. ERC 679 unchanged;
netlist nets/components identical.

Directive: hw-02
Tracker: #58

Co-Authored-By: Claude Opus 5.5 <noreply@anthropic.com>
Parts:
- C179, C44: Dielectric (none) -> unspecified; Tolerance (none) -> unspecified; Voltage (none) -> >=6.3 V (inferred: 3.3 V on 3V3A)
- C180: Dielectric (none) -> unspecified; Tolerance (none) -> unspecified; Voltage (none) -> >=6.3 V (inferred: 3.3 V on Net-(U14-BSPLY))
- C42, C46: Dielectric (none) -> unspecified; Status (none) -> needs-David: see docs/hardware/fmcw3 memo; Tolerance (none) -> unspecified; Voltage (none) -> >=6.3 V (inferred: 3 V on Net-(U9-RFOUT))
- C48: Dielectric (none) -> unspecified; Status (none) -> needs-David: see docs/hardware/fmcw3 memo; Tolerance (none) -> unspecified; Voltage (none) -> >=6.3 V (inferred default: no supply rail on these nets)
- C49: Dielectric (none) -> unspecified; Tolerance (none) -> unspecified; Voltage (none) -> >=6.3 V (inferred: 3.6 V on 3V6)
- FB5, FB6: DigiKey PN (none) -> 490-5263-1-ND; MPN (none) -> BLM18PG181SN1D; Manufacturer (none) -> Murata Electronics
- L1: DigiKey PN (none) -> 490-7690-1-ND; MPN (none) -> LQW15AN9N9J80D; Manufacturer (none) -> Murata Electronics
- L2: Status (none) -> needs-David: see docs/hardware/fmcw3 memo; Tolerance (none) -> unspecified
- P1: DigiKey PN (none) -> CONSMA003.062-ND; MPN (none) -> CONSMA003.062; Manufacturer (none) -> TE Connectivity Linx
- R22: Tolerance (none) -> unspecified
- U11: DigiKey PN (none) -> 863-1398-1-ND; MPN (none) -> SKY65404-31; Manufacturer (none) -> Skyworks Solutions Inc.
- U9: DigiKey PN (none) -> 296-48786-1-ND; MPN (none) -> TRF37A73IDSGR; Manufacturer (none) -> Texas Instruments
