File: hardware/tx.kicad_sch (KiCad schematic)
At the start: 54 parts, among them Q1 RE1C002UN, U1 ADF4158, U10 HMC431LP4, U12 PAT1220-6dB, U14 MGA-25203, U15 SMA, U3 PAT1220-6dB, U7 TLV172DCK

Commit message: Hardware: apply sourcing fields to fmcw3 schematic symbols (hw-02)
Adds Manufacturer, MPN, DigiKey PN, Status (obsolete/NFND/needs-David:
see docs/hardware/fmcw3 memo) and, for generic passives, spec-only
Tolerance/Voltage/Dielectric hidden fields to 355 refs from
parts/fields_to_apply.csv. The 4 existing manf# fields are renamed to
MPN. Value, footprint, nets and PCB untouched. ERC 679 unchanged;
netlist nets/components identical.

Directive: hw-02
Tracker: #58

Co-Authored-By: Claude Opus 5.5 <noreply@anthropic.com>
Parts:
- C10, C14, C29, C32, C33, C34, C36: Dielectric (none) -> unspecified; Tolerance (none) -> unspecified; Voltage (none) -> >=6.3 V (inferred default: no supply rail on these nets)
- C11, C8: Dielectric (none) -> unspecified; Status (none) -> needs-David: see docs/hardware/fmcw3 memo; Tolerance (none) -> unspecified; Voltage (none) -> >=6.3 V (inferred default: no supply rail on these nets)
- C176, C2, C26, C38, C4, C43: Dielectric (none) -> unspecified; Tolerance (none) -> unspecified; Voltage (none) -> >=6.3 V (inferred: 3.6 V on 3V6)
- C21: Dielectric (none) -> unspecified; Tolerance (none) -> unspecified; Voltage (none) -> >=16 V (inferred: 10 V on 10V)
- C28, C3, C5: Dielectric (none) -> unspecified; Tolerance (none) -> unspecified; Voltage (none) -> >=6.3 V (inferred: 3.3 V on 3V3A)
- C39, C40, C41: Dielectric (none) -> unspecified; Tolerance (none) -> unspecified; Voltage (none) -> >=6.3 V (inferred: 3.3 V on Net-(U14-BSPLY))
- C6, C7: Dielectric (none) -> unspecified; Tolerance (none) -> unspecified; Voltage (none) -> >=10 V (inferred: 5 V on Net-(U1-VP))
- FB2, FB3: DigiKey PN (none) -> 490-5263-1-ND; MPN (none) -> BLM18PG181SN1D; Manufacturer (none) -> Murata Electronics
- FB4: DigiKey PN (none) -> 1276-6374-2-ND; MPN (none) -> CIC21P101NE; Manufacturer (none) -> Samsung Electro-Mechanics; Status (none) -> Obsolete: see docs/hardware/fmcw3 memo
- Q1: DigiKey PN (none) -> RE1C002UNTCLCT-ND; MPN (none) -> RE1C002UNTCL; Manufacturer (none) -> Rohm Semiconductor
- R1, R10, R14, R18, R39, R4, R5, R6, R7: Tolerance (none) -> unspecified
- R11, R12, R17, R9: Status (none) -> needs-David: see docs/hardware/fmcw3 memo; Tolerance (none) -> unspecified
- U1: DigiKey PN (none) -> 505-ADF4158CCPZ-ND; MPN (none) -> ADF4158CCPZ; Manufacturer (none) -> Analog Devices Inc.; manf# ADF4158CCPZ -> (none)
- U10: DigiKey PN (none) -> 1127-1036-1-ND; MPN (none) -> HMC431LP4ETR; Manufacturer (none) -> Analog Devices Inc.; manf# HMC431LP4ETR -> (none)
- U12, U3: DigiKey PN (none) -> PAT126CT-ND; MPN (none) -> PAT1220-C-6DB-T5; Manufacturer (none) -> Susumu
- U14: DigiKey PN (none) -> 516-2289-ND; MPN (none) -> MGA-25203-BLKG; Manufacturer (none) -> Broadcom Limited; Status (none) -> Obsolete: see docs/hardware/fmcw3 memo; manf# MGA-25203-BLKG -> (none)
- U15: DigiKey PN (none) -> CONSMA003.062-ND; MPN (none) -> CONSMA003.062; Manufacturer (none) -> TE Connectivity Linx; manf# CONSMA003.062 -> (none)
- U7: DigiKey PN (none) -> 296-48697-1-ND; MPN (none) -> TLV172IDCKR; Manufacturer (none) -> Texas Instruments
