File: hardware/usb.kicad_sch (KiCad schematic)
At the start: 33 parts, among them U31 USB-MICRO, U32 93LC46B, U33 FT2232H, Y1 ABM10-167-12.000MHZ-T3

Commit message: Hardware: apply sourcing fields to fmcw3 schematic symbols (hw-02)
Adds Manufacturer, MPN, DigiKey PN, Status (obsolete/NFND/needs-David:
see docs/hardware/fmcw3 memo) and, for generic passives, spec-only
Tolerance/Voltage/Dielectric hidden fields to 355 refs from
parts/fields_to_apply.csv. The 4 existing manf# fields are renamed to
MPN. Value, footprint, nets and PCB untouched. ERC 679 unchanged;
netlist nets/components identical.

Directive: hw-02
Tracker: #58

Co-Authored-By: Claude Opus 5.5 <noreply@anthropic.com>
Parts:
- C152, C153, C154, C158, C159, C160, C161, C207, C210, C211, C212: Dielectric (none) -> unspecified; Tolerance (none) -> unspecified; Voltage (none) -> >=6.3 V (inferred: 3.6 V on 3V6)
- C155, C156, C157: Dielectric (none) -> unspecified; Tolerance (none) -> unspecified; Voltage (none) -> >=6.3 V (inferred: 3.3 V on Net-(U33-VPHY))
- C208, C209: Dielectric (none) -> unspecified; Tolerance (none) -> unspecified; Voltage (none) -> >=6.3 V (inferred default: no supply rail on these nets)
- FB12, FB14: DigiKey PN (none) -> 490-5263-1-ND; MPN (none) -> BLM18PG181SN1D; Manufacturer (none) -> Murata Electronics
- R71, R72, R73, R79, R80, R81, R82, R83, R84, R85, R88: Tolerance (none) -> unspecified
- U31: Status (none) -> needs-David: see docs/hardware/fmcw3 memo
- U32: DigiKey PN (none) -> 93LC46BT-I/OTCT-ND; MPN (none) -> 93LC46BT-I/OT; Manufacturer (none) -> Microchip Technology
- U33: DigiKey PN (none) -> 768-1024-1-ND; MPN (none) -> FT2232HL-REEL; Manufacturer (none) -> FTDI, Future Technology Devices International Ltd
- Y1: DigiKey PN (none) -> 535-13521-1-ND; MPN (none) -> ABM10-167-12.000MHZ-T3; Manufacturer (none) -> Abracon LLC
